File: KiCAD/_autosave-motee.kicad_pcb (KiCad board)
At the start: 2 copper layers, 49 parts, among them IC1 ATTINY841-MU, J1 SN65HVD3082EDGK, J2 drv8850, U1 TLE4946-2K, U10 pad, U11 pad, U12 pad, U13 pad, U14 pad, U15 pad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

Commit message: poprawki
Routing:
- net +3V3: track 89.3 -> 88.5 mm
