File: KiCAD/motee.sch (KiCad schematic (older format))
At the start: 49 parts, among them IC1 ATTINY841-MU, J1 SN65HVD3082EDGK, J2 drv8850, U1 TLE4946-2K, U10 pad, U11 pad, U12 pad, U13 pad, U14 pad, U15 pad, U16 pad, U17 MISO, U18 SCK, U19 RESET, U2 TLE4946-2K, U20 pad, U21 MOSI, U22 pad, U23 pad, U24 pad, U25 pad, U26 pad, U27 pad, U28 pad, U29 pad, U3 pad_round, U30 pad, U31 pad, U32 pad, U4 pad_round, U5 pad, U6 pad, U7 pad, U8 pad, U9 pad

Commit message: poprawki
Parts:
- IC1: footprint Housings_DFN_QFN:QFN-20-1EP_5x5mm_Pitch0.65mm -> kicad-libraries-master:QFN20-3X3
- U1, U2: footprint TO_SOT_Packages_SMD:SOT-23 -> kicad-libraries-master:SC59
Changed lines of the file:
@@
 LIBS:TLE4946-2K
 LIBS:pad
-LIBS:motee-cache
 EELAYER 25 0
 EELAYER END
@@
 F 0 "IC1" H 5850 3200 50  0000 C CNN
 F 1 "ATTINY841-MU" H 7400 1700 50  0000 C CNN
-F 2 "Housings_DFN_QFN:QFN-20-1EP_5x5mm_Pitch0.65mm" H 6700 2250 50  0000 C CIN
+F 2 "kicad-libraries-master:QFN20-3X3" H 6700 2250 50  0000 C CIN
 F 3 "" H 6700 2450 50  0000 C CNN
 	1    6700 2450
@@
 F 0 "U1" H 8300 4500 60  0000 C CNN
 F 1 "TLE4946-2K" H 8400 3850 60  0000 C CNN
-F 2 "TO_SOT_Packages_SMD:SOT-23" H 8400 3850 60  0000 C CNN
+F 2 "kicad-libraries-master:SC59" H 8400 3850 60  0000 C CNN
 F 3 "" H 8400 3850 60  0000 C CNN
 	1    8300 4200
@@
 F 0 "U2" H 8300 5300 60  0000 C CNN
 F 1 "TLE4946-2K" H 8400 4650 60  0000 C CNN
-F 2 "TO_SOT_Packages_SMD:SOT-23" H 8400 4650 60  0000 C CNN
+F 2 "kicad-libraries-master:SC59" H 8400 4650 60  0000 C CNN
 F 3 "" H 8400 4650 60  0000 C CNN
 	1    8300 5000

Commit message: poprawiona
Parts:
- U1, U2: footprint kicad-libraries-master:SC59 -> TO_SOT_Packages_SMD:SOT-23
Connections:
- net DIR: no longer U18.1
- net IN1L: now also U18.1
- net nSLEEP: now also D1.2 (A), R7.2
Other:
- moved on the sheet: R7
Changed lines of the file:
@@
 LIBS:TLE4946-2K
 LIBS:pad
+LIBS:motee-cache
 EELAYER 25 0
 EELAYER END
@@
 Text GLabel 4150 1850 2    60   Input ~ 0
 OUT1
-Text GLabel 4300 2550 2    60   Input ~ 0
-nSLEEP
 $Comp
 L R R5
 U 1 1 56E9C558
 P 4200 2450
-F 0 "R5" V 4280 2450 50  0000 C CNN
-F 1 "2.4K" V 4200 2450 50  0000 C CNN
+F 0 "R5" V 4150 2300 50  0000 C CNN
+F 1 "2.4K" V 4100 2450 50  0000 C CNN
 F 2 "Resistors_SMD:R_0402" V 4130 2450 50  0001 C CNN
 F 3 "" H 4200 2450 50  0000 C CNN
@@
 	4500 2450 4350 2450
 Wire Wire Line
-	4000 2550 4300 2550
-Wire Wire Line
 	4000 2750 4300 2750
 Wire Wire Line
@@
 Wire Wire Line
 	7750 2850 8000 2850
-Wire Wire Line
-	7750 2750 8000 2750
 Wire Wire Line
 	7750 2550 8000 2550
@@
 F 0 "U1" H 8300 4500 60  0000 C CNN
 F 1 "TLE4946-2K" H 8400 3850 60  0000 C CNN
-F 2 "kicad-libraries-master:SC59" H 8400 3850 60  0000 C CNN
+F 2 "TO_SOT_Packages_SMD:SOT-23" H 8400 3850 60  0000 C CNN
 F 3 "" H 8400 3850 60  0000 C CNN
 	1    8300 4200
@@
 F 0 "U2" H 8300 5300 60  0000 C CNN
 F 1 "TLE4946-2K" H 8400 4650 60  0000 C CNN
-F 2 "kicad-libraries-master:SC59" H 8400 4650 60  0000 C CNN
+F 2 "TO_SOT_Packages_SMD:SOT-23" H 8400 4650 60  0000 C CNN
 F 3 "" H 8400 4650 60  0000 C CNN
 	1    8300 5000
@@
 L R R7
 U 1 1 56EE0EF1
-P 8150 2750
-F 0 "R7" V 8230 2750 50  0000 C CNN
-F 1 "220R" H 8150 2750 50  0000 R CNN
-F 2 "Resistors_SMD:R_0402" V 8080 2750 50  0001 C CNN
-F 3 "" H 8150 2750 50  0000 C CNN
-	1    8150 2750
+P 8000 2750
+F 0 "R7" V 8080 2750 50  0000 C CNN
+F 1 "220R" H 8000 2750 50  0000 R CNN
+F 2 "Resistors_SMD:R_0402" V 7930 2750 50  0001 C CNN
+F 3 "" H 8000 2750 50  0000 C CNN
+	1    8000 2750
 	0    -1   -1   0
 $EndComp
@@
 $EndComp
 Wire Wire Line
-	8300 2750 8350 2750
+	8150 2750 8350 2750
 Wire Wire Line
 	8750 2750 8750 2850
@@
 RESET
 Text GLabel 1700 5950 0    60   Input ~ 0
-DIR
+IN1L
 $Comp
 L +3.3V #PWR025
@@
 	6150 5150 6650 5150
 Connection ~ 6650 5250
+Wire Wire Line
+	4000 2550 4400 2550
+Wire Wire Line
+	7850 2750 7750 2750
+Wire Wire Line
+	8250 2750 8250 2600
+Wire Wire Line
+	8250 2600 8500 2600
+Connection ~ 8250 2750
+Text GLabel 8500 2600 2    60   Input ~ 0
+nSLEEP
+Text GLabel 4400 2550 2    60   Input ~ 0
+nSLEEP
 $EndSCHEMATC
