File: KiCAD/motee.kicad_pcb (KiCad board)
At the start: 2 copper layers, 49 parts, among them IC1 ATTINY841-MU, J1 SN65HVD3082EDGK, J2 drv8850, U1 TLE4946-2K, U10 pad, U11 pad, U12 pad, U13 pad, U14 pad, U15 pad, U16 pad, U17 MISO, U18 SCK, U19 RESET, U2 TLE4946-2K, U20 pad, U21 MOSI, U22 pad, U23 pad, U24 pad, U25 pad, U26 pad, U27 pad, U28 pad, U29 pad, U3 pad_round, U30 pad, U31 pad, U32 pad, U4 pad_round, U5 pad, U6 pad, U7 pad, U8 pad, U9 pad

Commit message: poprawiona
Parts:
- U1, U2: footprint kicad-libraries-master:SOT23-3 -> TO_SOT_Packages_SMD:SOT-23
- turned U1 to 240 degrees
- turned U2 to 300 degrees
Connections:
- D1 pad 2: Net-(D1-Pad2) -> nSLEEP
- J2 pad 9: (no net) -> nSLEEP
- R7 pad 2: Net-(D1-Pad2) -> nSLEEP
- U18 pad 1: DIR -> IN1L
Routing:
- net DIR: track 48.6 -> 20.2 mm, vias 1 -> 0
- net IN1L: track 11.0 -> 30.1 mm, vias 0 -> 1
- net nSLEEP: track 0.00 -> 19.0 mm
- net Net-(D1-Pad2): track 2.67 -> 0.00 mm
- net IN1H: track 38.8 -> 40.6 mm
- net +3V3: track 89.3 -> 88.5 mm
- net IN2H: track 21.8 -> 22.3 mm

Commit message: gerbery
Parts:
- moved U29 16.2 mm to (34.5, 176.6), turned to 270 degrees
- moved U7 16.2 mm to (34.5, 176.6), turned to 270 degrees
- moved U10 16.0 mm to (34.5, 163.3), turned to 270 degrees
- moved U32 15.9 mm to (34.5, 163.3), turned to 270 degrees
- moved U28 12.3 mm to (34.5, 173.9), turned to 270 degrees
- moved U6 12.3 mm to (34.5, 173.9), turned to 270 degrees
- moved U31 12.1 mm to (34.5, 165.9), turned to 270 degrees
- moved U9 12.1 mm to (34.5, 165.9), turned to 270 degrees
- moved U1 10.1 mm to (42.5, 173.5), turned to 60 degrees
- moved U27 9.51 mm to (34.5, 171.2), turned to 270 degrees
- moved U30 9.51 mm to (34.5, 168.6), turned to 270 degrees
- moved U5 9.51 mm to (34.5, 171.2), turned to 270 degrees
- moved U8 9.51 mm to (34.5, 168.6), turned to 270 degrees
- moved U2 8.91 mm to (42.5, 167.0), turned to 120 degrees
- moved U4 8.13 mm to (39.4, 173.9), turned to 270 degrees
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
Commit message: gerbery_v2
Parts:
- moved R5 0.40 mm to (61.2, 171.9)
- moved R7 0.05 mm to (67.3, 170.1)
Routing:
- net nSLEEP: track 19.0 -> 23.6 mm, vias 0 -> 2
- net GND: track 116.6 -> 115.1 mm, vias 7 -> 8
Other:
- net class Default: clearance 0.1 -> 0.2
- net class one: clearance 0.1 -> 0.2
- rule trace_clearance: 0.1 -> 0.2
