File: motee_v3/KiCAD/motee_v3.sch (KiCad schematic (older format))
At the start: 58 parts, among them J1 SN65HVD3082EDGK, U1 STM32F103, U10 pad, U11 pad, U12 pad, U13 pad, U14 pad, U15 pad, U16 pad, U17 pad, U18 pad, U19 pad, U2 DRV8801, U20 pad, U21 pad, U22 pad, U23 pad, U24 pad, U25 pad, U26 pad, U27 pad, U28 pad, U29 pad, U3 TLE4946-2K, U30 pad, U31 pad, U32 pad, U33 pad, U34 pad, U4 TLE4946-2K, U5 pad_round, U6 pad_round, U7 micro-usb, U8 LP38693, U9 LP38693

Commit message: poprawki
Parts:
- C3: value C_Small -> 100nF
- L1: value L_Small -> 10uH
Changed lines of the file:
@@
 P 5050 3650
 F 0 "L1" H 5080 3690 50  0000 L CNN
-F 1 "L_Small" H 5080 3610 50  0000 L CNN
+F 1 "10uH" H 5080 3610 50  0000 L CNN
 F 2 "SMD_Packages:SMD-1206_Pol" H 5050 3650 50  0001 C CNN
 F 3 "" H 5050 3650 50  0000 C CNN
@@
 P 5200 3750
 F 0 "C3" H 5210 3820 50  0000 L CNN
-F 1 "C_Small" H 5200 3650 50  0000 L CNN
+F 1 "100nF" H 5200 3650 50  0000 L CNN
 F 2 "Capacitors_SMD:C_0402" H 5200 3750 50  0001 C CNN
 F 3 "" H 5200 3750 50  0000 C CNN

Commit message: rezystor i dioda 0805
Parts:
- D1: footprint LEDs:LED_0402 -> LEDs:LED_0603
- L1: footprint SMD_Packages:SMD-1206_Pol -> Inductors_NEOSID:Neosid_Inductor_SM0603CG
- R1: footprint Resistors_SMD:R_0402 -> Resistors_SMD:R_0603
Changed lines of the file:
@@
 F 0 "L1" H 5080 3690 50  0000 L CNN
 F 1 "10uH" H 5080 3610 50  0000 L CNN
-F 2 "SMD_Packages:SMD-1206_Pol" H 5050 3650 50  0001 C CNN
+F 2 "Inductors_NEOSID:Neosid_Inductor_SM0603CG" H 5050 3650 50  0001 C CNN
 F 3 "" H 5050 3650 50  0000 C CNN
 	1    5050 3650
@@
 F 0 "R1" V 2530 2200 50  0000 C CNN
 F 1 "0.2 R" V 2450 2200 50  0000 C CNN
-F 2 "Resistors_SMD:R_0402" V 2380 2200 50  0001 C CNN
+F 2 "Resistors_SMD:R_0603" V 2380 2200 50  0001 C CNN
 F 3 "" H 2450 2200 50  0000 C CNN
 	1    2450 2200
@@
 F 0 "D1" H 7300 2700 50  0000 C CNN
 F 1 "LED" H 7300 2500 50  0000 C CNN
-F 2 "LEDs:LED_0402" H 7300 2600 50  0001 C CNN
+F 2 "LEDs:LED_0603" H 7300 2600 50  0001 C CNN
 F 3 "" H 7300 2600 50  0000 C CNN
 	1    7300 2600

Commit message: wylane masy i boot0
Connections:
- net GND: now also U1.35 (BOOT0)
Changed lines of the file:
@@
+	1    0    0    -1
+$EndComp
+$Comp
+L GND #PWR?
+U 1 1 57EDA377
+P 5750 4000
+F 0 "#PWR?" H 5750 3750 50  0001 C CNN
+F 1 "GND" H 5750 3850 50  0000 C CNN
+F 2 "" H 5750 4000 50  0000 C CNN
+F 3 "" H 5750 4000 50  0000 C CNN
+	1    5750 4000
 	1    0    0    -1
 $EndComp

Commit message: bug fixes
Parts:
- added C13, C5: 22pF, Capacitors_SMD:C_0402, symbol C_Small
- added R11: 1k, Resistors_SMD:R_0402, symbol R
- added Y1: Crystal_GND24, Crystals:Crystal_SMD_SeikoEpson_FA238-4pin_3.2x2.5mm, symbol Crystal_GND24
- D1: symbol LED -> LED-RESCUE-motee_v3
Connections:
- wire segments 123 -> 136
Other:
- moved on the sheet: C11, C12, R8, R9
Changed lines of the file:
@@
 EESchema Schematic File Version 2
+LIBS:motee_v3-rescue
 LIBS:power
 LIBS:device
@@
 P 4900 3600
 F 0 "#PWR05" H 4900 3450 50  0001 C CNN
-F 1 "+3.3V" H 4900 3740 50  0000 C CNN
+F 1 "+3.3V" H 4750 3550 50  0000 C CNN
 F 2 "" H 4900 3600 50  0000 C CNN
 F 3 "" H 4900 3600 50  0000 C CNN
@@
 U 1 1 577A71BE
 P 5050 3650
-F 0 "L1" H 5080 3690 50  0000 L CNN
-F 1 "10uH" H 5080 3610 50  0000 L CNN
+F 0 "L1" V 5000 3650 50  0000 L CNN
+F 1 "10uH" V 5100 3550 50  0000 L CNN
 F 2 "Inductors_NEOSID:Neosid_Inductor_SM0603CG" H 5050 3650 50  0001 C CNN
 F 3 "" H 5050 3650 50  0000 C CNN
@@
 U 1 1 577A7A9A
 P 5200 3750
-F 0 "C3" H 5210 3820 50  0000 L CNN
-F 1 "100nF" H 5200 3650 50  0000 L CNN
+F 0 "C3" H 5050 3700 50  0000 L CNN
+F 1 "100nF" H 4950 3600 50  0000 L CNN
 F 2 "Capacitors_SMD:C_0402" H 5200 3750 50  0001 C CNN
 F 3 "" H 5200 3750 50  0000 C CNN
@@
 L R R9
 U 1 1 577CFCE2
-P 10100 5350
-F 0 "R9" V 10180 5350 50  0000 C CNN
-F 1 "1k" V 10100 5350 50  0000 C CNN
-F 2 "Resistors_SMD:R_0402" V 10030 5350 50  0001 C CNN
-F 3 "" H 10100 5350 50  0000 C CNN
-	1    10100 5350
-	-1   0    0    1
+P 10100 5625
+F 0 "R9" V 10180 5625 50  0000 C CNN
+F 1 "1k" V 10100 5625 50  0000 C CNN
+F 2 "Resistors_SMD:R_0402" V 10030 5625 50  0001 C CNN
+F 3 "" H 10100 5625 50  0000 C CNN
+	1    10100 5625
+	0    1    1    0
 $EndComp
 $Comp
@@
 L CP1_Small C12
 U 1 1 577D4BB9
-P 10300 5300
-F 0 "C12" H 10310 5370 50  0000 L CNN
-F 1 "1uF" H 10310 5220 50  0000 L CNN
-F 2 "Capacitors_SMD:C_1206" H 10300 5300 50  0001 C CNN
-F 3 "" H 10300 5300 50  0000 C CNN
-	1    10300 5300
+P 10100 5300
+F 0 "C12" H 10110 5370 50  0000 L CNN
+F 1 "1uF" H 10110 5220 50  0000 L CNN
+F 2 "Capacitors_SMD:C_1206" H 10100 5300 50  0001 C CNN
+F 3 "" H 10100 5300 50  0000 C CNN
+	1    10100 5300
 	1    0    0    -1
 $EndComp
@@
 L GND #PWR022
 U 1 1 577D5240
-P 10300 5500
-F 0 "#PWR022" H 10300 5250 50  0001 C CNN
-F 1 "GND" H 10300 5350 50  0000 C CNN
-F 2 "" H 10300 5500 50  0000 C CNN
-F 3 "" H 10300 5500 50  0000 C CNN
-	1    10300 5500
+P 10100 5400
+F 0 "#PWR022" H 10100 5150 50  0001 C CNN
+F 1 "GND" H 10100 5250 50  0000 C CNN
+F 2 "" H 10100 5400 50  0000 C CNN
+F 3 "" H 10100 5400 50  0000 C CNN
+	1    10100 5400
 	1    0    0    -1
 $EndComp
@@
 $EndComp
 Connection ~ 5650 2400
-Wire Wire Line
-	9950 5500 10100 5500
 Connection ~ 9950 5200
 Wire Wire Line
@@
 Wire Wire Line
 	5750 3900 5700 3900
-Connection ~ 10100 5200
 Wire Wire Line
 	5650 2300 5650 2500
@@
 Wire Wire Line
 	10300 5200 10300 5150
-Wire Wire Line
-	10300 5400 10300 5500
 Connection ~ 10300 5200
 Wire Wire Line
@@
 Wire Wire Line
 	5550 2700 5550 2750
-Text GLabel 5400 5100 2    60   Input ~ 0
+Text GLabel 5850 4900 2    60   Input ~ 0
 VBUS
-Text GLabel 5400 5200 2    60   Input ~ 0
+Text GLabel 5800 5200 2    60   Input ~ 0
 D+
-Text GLabel 5400 5300 2    60   Input ~ 0
+Text GLabel 5425 5300 2    60   Input ~ 0
 D-
 $Comp
@@
 L R R8
 U 1 1 578FDA35
-P 10100 3950
-F 0 "R8" V 10180 3950 50  0000 C CNN
-F 1 "1k" V 10100 3950 50  0000 C CNN
-F 2 "Resistors_SMD:R_0402" V 10030 3950 50  0001 C CNN
-F 3 "" H 10100 3950 50  0000 C CNN
-	1    10100 3950
-	-1   0    0    1
+P 10125 4225
+F 0 "R8" V 10205 4225 50  0000 C CNN
+F 1 "1k" V 10125 4225 50  0000 C CNN
+F 2 "Resistors_SMD:R_0402" V 10055 4225 50  0001 C CNN
+F 3 "" H 10125 4225 50  0000 C CNN
+	1    10125 4225
+	0    -1   -1   0
 $EndComp
 $Comp
@@
 L CP1_Small C11
 U 1 1 578FDA47
-P 10300 3900
-F 0 "C11" H 10310 3970 50  0000 L CNN
-F 1 "1uF" H 10310 3820 50  0000 L CNN
-F 2 "Capacitors_Tantalum_SMD:TantalC_SizeT_EIA-3528" H 10300 3900 50  0001 C CNN
-F 3 "" H 10300 3900 50  0000 C CNN
-	1    10300 3900
+P 10100 3900
+F 0 "C11" H 10110 3970 50  0000 L CNN
+F 1 "1uF" H 10110 3820 50  0000 L CNN
+F 2 "Capacitors_Tantalum_SMD:TantalC_SizeT_EIA-3528" H 10100 3900 50  0001 C CNN
+F 3 "" H 10100 3900 50  0000 C CNN
+	1    10100 3900
 	1    0    0    -1
 $EndComp
@@
 L GND #PWR028
 U 1 1 578FDA4D
-P 10300 4100
-F 0 "#PWR028" H 10300 3850 50  0001 C CNN
-F 1 "GND" H 10300 3950 50  0000 C CNN
-F 2 "" H 10300 4100 50  0000 C CNN
-F 3 "" H 10300 4100 50  0000 C CNN
-	1    10300 4100
+P 10100 4000
+F 0 "#PWR028" H 10100 3750 50  0001 C CNN
+F 1 "GND" H 10100 3850 50  0000 C CNN
+F 2 "" H 10100 4000 50  0000 C CNN
+F 3 "" H 10100 4000 50  0000 C CNN
+	1    10100 4000
 	1    0    0    -1
 $EndComp
@@
 	1    0    0    -1
 $EndComp
-Wire Wire Line
-	9950 4100 10100 4100
 Connection ~ 9950 3800
 Wire Wire Line
@@
 Wire Wire Line
 	10300 3800 10300 3750
-Wire Wire Line
-	10300 4000 10300 4100
 Connection ~ 10300 3800
 Wire Wire Line
@@
 $EndComp
 Wire Wire Line
-	5300 5100 5400 5100
-Wire Wire Line
-	5300 5200 5400 5200
-Wire Wire Line
-	5300 5300 5400 5300
+	5300 5200 5800 5200
 Wire Wire Line
 	5300 5400 5400 5400
@@
 	2400 2350 2350 2350
 $Comp
-L LED D1
+L LED-RESCUE-motee_v3 D1
 U 1 1 57D88835
 P 7300 2600
@@
 $EndComp
 $Comp
-L GND #PWR?
+L GND #PWR035
 U 1 1 57EDA377
 P 5750 4000
-F 0 "#PWR?" H 5750 3750 50  0001 C CNN
+F 0 "#PWR035" H 5750 3750 50  0001 C CNN
 F 1 "GND" H 5750 3850 50  0000 C CNN
 F 2 "" H 5750 4000 50  0000 C CNN
@@
 	1    0    0    -1
 $EndComp
+$Comp
+L C_Small C13
+U 1 1 587906A1
+P 5250 3550
+F 0 "C13" H 5260 3620 50  0000 L CNN
+F 1 "22pF" V 5300 3650 50  0000 L CNN
+F 2 "Capacitors_SMD:C_0402" H 5250 3550 50  0001 C CNN
+F 3 "" H 5250 3550 50  0000 C CNN
+	1    5250 3550
+	0    1    1    0
+$EndComp
+$Comp
+L C_Small C5
+U 1 1 58790797
+P 5250 3250
+F 0 "C5" H 5260 3320 50  0000 L CNN
+F 1 "22pF" V 5150 3150 50  0000 L CNN
+F 2 "Capacitors_SMD:C_0402" H 5250 3250 50  0001 C CNN
+F 3 "" H 5250 3250 50  0000 C CNN
+	1    5250 3250
+	0    1    1    0
+$EndComp
+Wire Wire Line
+	5150 3250 5150 3550
+$Comp
+L GND #PWR036
+U 1 1 587912D3
+P 5025 3425
+F 0 "#PWR036" H 5025 3175 50  0001 C CNN
+F 1 "GND" H 4925 3425 50  0000 C CNN
+F 2 "" H 5025 3425 50  0000 C CNN
+F 3 "" H 5025 3425 50  0000 C CNN
+	1    5025 3425
+	1    0    0    -1
+$EndComp
+Wire Wire Line
+	5145 3445 5145 3455
+Wire Wire Line
+	9950 5500 9950 5625
+Text GLabel 10325 5625 2    60   Input ~ 0
+VBUS
+Wire Wire Line
+	10250 5625 10325 5625
+Connection ~ 10100 5200
+Wire Wire Line
+	9950 4100 9950 4225
+Wire Wire Line
+	9950 4225 9975 4225
+Wire Wire Line
+	10275 4225 10350 4225
+$Comp
+L R R11
+U 1 1 587A28E8
+P 5725 5050
+F 0 "R11" V 5805 5050 50  0000 C CNN
+F 1 "1k" V 5725 5050 50  0000 C CNN
+F 2 "Resistors_SMD:R_0402" V 5655 5050 50  0001 C CNN
+F 3 "" H 5725 5050 50  0000 C CNN
+	1    5725 5050
+	1    0    0    -1
+$EndComp
+$Comp
+L +8V #PWR037
+U 1 1 587A4FD8
+P 10350 4225
+F 0 "#PWR037" H 10350 4075 50  0001 C CNN
+F 1 "+8V" H 10350 4365 50  0000 C CNN
+F 2 "" H 10350 4225 50  0000 C CNN
+F 3 "" H 10350 4225 50  0000 C CNN
+	1    10350 4225
+	1    0    0    -1
+$EndComp
+Wire Wire Line
+	5350 3250 5750 3250
+Wire Wire Line
+	5750 3250 5750 3400
+Wire Wire Line
+	5750 3550 5750 3500
+Wire Wire Line
+	5350 3550 5750 3550
+Wire Wire Line
+	5425 3550 5425 3525
+Connection ~ 5425 3250
+Wire Wire Line
+	5025 3400 5225 3400
+Connection ~ 5150 3400
+Wire Wire Line
+	5625 3400 5625 3425
+$Comp
+L GND #PWR038
+U 1 1 587A78B2
+P 5625 3425
+F 0 "#PWR038" H 5625 3175 50  0001 C CNN
+F 1 "GND" H 5525 3425 50  0000 C CNN
+F 2 "" H 5625 3425 50  0000 C CNN
+F 3 "" H 5625 3425 50  0000 C CNN
+	1    5625 3425
+	1    0    0    -1
+$EndComp
+Wire Wire Line
+	5025 3400 5025 3425
+Wire Wire Line
+	5300 5100 5575 5100
+Wire Wire Line
+	5575 5100 5575 4900
+Wire Wire Line
+	5575 4900 5850 4900
+Connection ~ 5725 4900
+Connection ~ 5725 5200
+Wire Wire Line
+	5300 5300 5425 5300
+Connection ~ 5425 3550
+$Comp
+L Crystal_GND24 Y1
+U 1 1 587AB9ED
+P 5425 3400
+F 0 "Y1" H 5550 3600 50  0000 L CNN
+F 1 "Crystal_GND24" H 5550 3525 50  0000 L CNN
+F 2 "Crystals:Crystal_SMD_SeikoEpson_FA238-4pin_3.2x2.5mm" H 5425 3400 50  0001 C CNN
+F 3 "" H 5425 3400 50  0000 C CNN
+	1    5425 3400
+	0    1    1    0
+$EndComp
 $EndSCHEMATC
